File: hardware/kicad/SQMeter-Hardware-Zero.kicad_sch (KiCad schematic)
At the start: 46 parts, among them J1 12V IN, J10 AUX, J11 Zero left, J12 Zero right, J3 I2C TSL2591, J4 I2C MLX90614, J5 I2C BME280, J6 I2C SPARE, J7 GPS, J8 RG-15, J9 WIND, Q1 AO3401A, U1 AP63205WU, U4 USBLC6-2SC6, U5 USBLC6-2SC6, U6 USBLC6-2SC6

Commit message: feat: second I2C bus for a second TSL2591 (SQM + SQM-L)
TSL2591 has a fixed address, so the second sensor gets its own bus on
GPIO10/11 (I2C-2 JST-XH port, own pull-ups and ESD). AUX drops to IO6/IO7.
Q1 gate zener replaced by a resistor divider (one fewer extended part).
Parts:
- removed D2: BZT52C10, Diode_SMD:D_SOD-123, symbol Device:D_Zener
- removed J10: AUX, Connector_JST:JST_XH_B6B-XH-A_1x06_P2.50mm_Vertical, symbol Connector_Generic:Conn_01x06
- added J10: AUX, Connector_JST:JST_XH_B4B-XH-A_1x04_P2.50mm_Vertical, symbol Connector_Generic:Conn_01x04
- added J13: I2C-2 TSL2591 #2, Connector_JST:JST_XH_B4B-XH-A_1x04_P2.50mm_Vertical, symbol Connector_Generic:Conn_01x04
- added R19: 10k, Resistor_SMD:R_0603_1608Metric, symbol Device:R
- added R20, R21: 4.7k, Resistor_SMD:R_0603_1608Metric, symbol Device:R
- added U7: USBLC6-2SC6, Package_TO_SOT_SMD:SOT-23-6, symbol Power_Protection:USBLC6-2SC6
- J3: value I2C TSL2591 -> I2C TSL2591 #1
Connections:
- net +12V: now also R19.1
- net +3V3: now also J10.2 (Pin_2), J13.2 (Pin_2), R20.1, R21.1, U7.5 (VBUS)
- net AUX1: now also J10.3 (Pin_3)
- net AUX2: now also J10.4 (Pin_4)
- net GND: now also J10.1 (Pin_1), J13.1 (Pin_1), U7.2 (GND)
- net Q1_G: now also R19.2
- net AUX3 renamed SDA2
- net SDA2: now also J13.3 (Pin_3), R20.2, U7.1 (I/O1), U7.6 (I/O1)
- net AUX4 renamed SCL2
- net SCL2: now also J13.4 (Pin_4), R21.2, U7.3 (I/O2), U7.4 (I/O2)
