File: hardware/kicad/SQMeter-Hardware.kicad_sch (KiCad schematic)
At the start: 62 parts, among them J1 12V IN, J10 AUX, J2 USB-C, J3 I2C TSL2591, J4 I2C MLX90614, J5 I2C BME280, J6 I2C SPARE, J7 GPS, J8 RG-15, J9 WIND, Q1 AO3401A, SW1 RESET, SW2 BOOT, U1 AP63203WU, U2 USBLC6-2SC6, U3 ESP32-S3-WROOM-1-N16R8, U4 USBLC6-2SC6, U5 USBLC6-2SC6, U6 USBLC6-2SC6

Commit message: feat: DevKitC-1 socket variant, verified LCSC parts, JLC fab exports
- SQM_VARIANT=devkit swaps the soldered module for ESP32-S3-DevKitC-1 sockets
  (header geometry from Espressif's DXF), 5 V buck feeding the DevKit 5V pin,
  antenna keepout and silkscreen outline
- every part has an in-stock LCSC number; polyfuses moved to 24 V parts
- export_jlc.sh writes gerber zip, BOM and CPL per variant
- build retries routing until DRC has no unconnected or dangling items
Parts:
- C1: footprint Capacitor_SMD:CP_Elec_8x10.5 -> Capacitor_SMD:CP_Elec_8x10; LCSC (none) -> C165636
- D1: LCSC (none) -> C78413
- D2: LCSC (none) -> C173431
- D4: LCSC C72043 -> C12624
- F1: value 1.5A -> 1.5A 24V; LCSC (none) -> C32404
- F2: value 0.5A -> 0.5A 24V; LCSC (none) -> C492011
- J1: LCSC (none) -> C3697
- J10: LCSC (none) -> C144397
- J8: LCSC (none) -> C5188297
- J9: LCSC (none) -> C5188298
- L1: value 4.7u 3A -> 4.7u 3.3A; footprint Inductor_SMD:L_Bourns_SRN6045TA -> Inductor_SMD:L_Sunlord_SWPA6045S; LCSC (none) -> C78804
Changed lines of the file:
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@@
     (rev "v1.0-draft")
     (company "SQMeter")
-    (comment 1 "ESP32-S3, 12 V input, JST-XH I2C ports")
+    (comment 1 "ESP32-S3-WROOM-1, 12 V input, JST-XH I2C ports")
   )
   (text
@@
     (property
       "Description"
-      "Pluggable 5.08 mm: 1 = +12 V, 2 = GND"
+      "Pluggable 5.08 mm (2EDGRC): 1 = +12 V, 2 = GND"
+      (at 36.83 33.02 0)
+      (effects
+        (font
+          (size 1.27 1.27)
+        )
+        (hide yes)
+      )
+    )
+    (property
+      "LCSC"
+      "C3697"
       (at 36.83 33.02 0)
       (effects
@@
     (property
       "Value"
-      "1.5A"
+      "1.5A 24V"
       (at 62.23 46.355 0)
       (effects
@@
     (property
       "Description"
-      ""
+      "SMD1812P150TF/24"
+      (at 59.69 46.99 0)
+      (effects
+        (font
+          (size 1.27 1.27)
+        )
+        (hide yes)
+      )
+    )
+    (property
+      "LCSC"
+      "C32404"
       (at 59.69 46.99 0)
       (effects
@@
       )
     )
+    (property
+      "LCSC"
+      "C78413"
+      (at 109.22 41.91 0)
+      (effects
+        (font
+          (size 1.27 1.27)
+        )
+        (hide yes)
+      )
+    )
     (pin
       "1"
@@
       )
     )
+    (property
+      "LCSC"
+      "C173431"
+      (at 35.56 76.2 0)
+      (effects
+        (font
+          (size 1.27 1.27)
+        )
+        (hide yes)
+      )
+    )
     (pin
       "1"
@@
     (property
       "Footprint"
-      "Capacitor_SMD:CP_Elec_8x10.5"
+      "Capacitor_SMD:CP_Elec_8x10"
       (at 133.35 82.55 0)
       (effects
@@
     (property
       "Description"
-      ""
+      "BXJ 105C low-ESR"
+      (at 133.35 82.55 0)
+      (effects
+        (font
+          (size 1.27 1.27)
+        )
+        (hide yes)
+      )
+    )
+    (property
+      "LCSC"
+      "C165636"
       (at 133.35 82.55 0)
       (effects
@@
     (property
       "Value"
-      "4.7u 3A"
+      "4.7u 3.3A"
       (at 133.35 114.935 0)
       (effects
@@
     (property
       "Footprint"
-      "Inductor_SMD:L_Bourns_SRN6045TA"
+      "Inductor_SMD:L_Sunlord_SWPA6045S"
       (at 130.81 115.57 0)
       (effects
@@
     (property
       "Description"
-      ""
+      "Sunlord SWPA6045S"
+      (at 130.81 115.57 0)
+      (effects
+        (font
+          (size 1.27 1.27)
+        )
+        (hide yes)
+      )
+    )
+    (property
+      "LCSC"
+      "C78804"
       (at 130.81 115.57 0)
       (effects
@@
     (property
       "Value"
-      "0.5A"
+      "0.5A 24V"
       (at 17.78 147.955 0)
       (effects
@@
     (property
       "Description"
-      "RG-15 supply"
+      "RG-15 supply, SMD1206P050TF/24"
+      (at 15.24 148.59 0)
+      (effects
+        (font
+          (size 1.27 1.27)
+        )
+        (hide yes)
+      )
+    )
+    (property
+      "LCSC"
+      "C492011"
       (at 15.24 148.59 0)
       (effects
@@
     (property
       "LCSC"
-      "C72043"
+      "C12624"
       (at 410.21 130.81 0)
       (effects
@@
     (property
       "Description"
-      "Pluggable 3.5 mm: 1 GND, 2 V+ (12 V), 3 RG TX, 4 RG RX"
+      "Pluggable 3.5 mm (15EDGRC): 1 GND, 2 V+ (12 V), 3 RG TX, 4 RG RX"
+      (at 259.08 327.66 0)
+      (effects
+        (font
+          (size 1.27 1.27)
+        )
+        (hide yes)
+      )
+    )
+    (property
+      "LCSC"
+      "C5188297"
       (at 259.08 327.66 0)
       (effects
@@
     (property
       "Description"
-      "Pluggable 3.5 mm: 1 SPD, 2 GND, 3 DIR, 4 GND, 5 3V3 (pot vane excitation)"
+      "Pluggable 3.5 mm (15EDGRC): 1 SPD, 2 GND, 3 DIR, 4 GND, 5 3V3 (pot vane excitation)"
+      (at 474.98 38.1 0)
+      (effects
+        (font
+          (size 1.27 1.27)
+        )
+        (hide yes)
+      )
+    )
+    (property
+      "LCSC"
+      "C5188298"
       (at 474.98 38.1 0)
       (effects
@@
       (at 474.98 134.62 0)
       (effects
+        (font
+          (size 1.27 1.27)
+        )
+        (hide yes)
+      )
+    )
+    (property
+      "LCSC"
+      "C144397"
+      (at 474.98 134.62 0)
+      (effects

Commit message: feat: Waveshare ESP32-S3-Zero socket variant and one GPIO map for all boards
- SQM_VARIANT=zero: ESP32-S3-Zero-M on 2x9 sockets (Waveshare pinout and
  drawing), same 5 V feed scheme as the DevKit variant
- GPIO map unified across module, DevKit and Zero (limited by the Zero's
  GPIO1-13 headers): RG-15 1/2, wind 4/5, I2C 8/9, GPS 12/13, AUX 6/7/10/11
- fab exports for all three
Connections:
- net GPS_RX: now also U3.21 (IO13); no longer U3.11 (IO18)
- net GPS_TX: now also U3.20 (IO12); no longer U3.10 (IO17)
- net RG_RX: now also U3.38 (IO2); no longer U3.9 (IO16)
- net RG_TX: now also U3.39 (IO1); no longer U3.8 (IO15)
Changed lines of the file:
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@@
     )
   )
-  (label
-    "RG_TX"
-    (at 254 99.06 180)
-    (effects
-      (font
-        (size 1.27 1.27)
-      )
-      (justify right bottom)
-    )
+  (no_connect
+    (at 254 99.06)
   )
-  (label
-    "RG_RX"
-    (at 254 101.6 180)
-    (effects
-      (font
-        (size 1.27 1.27)
-      )
-      (justify right bottom)
-    )
+  (no_connect
+    (at 254 101.6)
   )
-  (label
-    "GPS_TX"
-    (at 284.48 60.96 0)
-    (effects
-      (font
-        (size 1.27 1.27)
-      )
-      (justify left bottom)
-    )
+  (no_connect
+    (at 284.48 60.96)
   )
-  (label
-    "GPS_RX"
-    (at 284.48 63.5 0)
-    (effects
-      (font
-        (size 1.27 1.27)
-      )
-      (justify left bottom)
-    )
+  (no_connect
+    (at 284.48 63.5)
   )
   (label
@@
     )
   )
-  (no_connect
-    (at 254 91.44)
+  (label
+    "GPS_TX"
+    (at 254 91.44 180)
+    (effects
+      (font
+        (size 1.27 1.27)
+      )
+      (justify right bottom)
+    )
   )
-  (no_connect
-    (at 254 93.98)
+  (label
+    "GPS_RX"
+    (at 254 93.98 180)
+    (effects
+      (font
+        (size 1.27 1.27)
+      )
+      (justify right bottom)
+    )
   )
   (no_connect
@@
     )
   )
-  (no_connect
-    (at 254 66.04)
+  (label
+    "RG_RX"
+    (at 254 66.04 180)
+    (effects
+      (font
+        (size 1.27 1.27)
+      )
+      (justify right bottom)
+    )
   )
-  (no_connect
-    (at 254 63.5)
+  (label
+    "RG_TX"
+    (at 254 63.5 180)
+    (effects
+      (font
+        (size 1.27 1.27)
+      )
+      (justify right bottom)
+    )
   )
   (symbol

Commit message: feat: second I2C bus for a second TSL2591 (SQM + SQM-L)
TSL2591 has a fixed address, so the second sensor gets its own bus on
GPIO10/11 (I2C-2 JST-XH port, own pull-ups and ESD). AUX drops to IO6/IO7.
Q1 gate zener replaced by a resistor divider (one fewer extended part).
Parts:
- removed D2: BZT52C10, Diode_SMD:D_SOD-123, symbol Device:D_Zener
- removed J10: AUX, Connector_JST:JST_XH_B6B-XH-A_1x06_P2.50mm_Vertical, symbol Connector_Generic:Conn_01x06
- added J10: AUX, Connector_JST:JST_XH_B4B-XH-A_1x04_P2.50mm_Vertical, symbol Connector_Generic:Conn_01x04
- added J13: I2C-2 TSL2591 #2, Connector_JST:JST_XH_B4B-XH-A_1x04_P2.50mm_Vertical, symbol Connector_Generic:Conn_01x04
- added R19: 10k, Resistor_SMD:R_0603_1608Metric, symbol Device:R
- added R20, R21: 4.7k, Resistor_SMD:R_0603_1608Metric, symbol Device:R
- added U7: USBLC6-2SC6, Package_TO_SOT_SMD:SOT-23-6, symbol Power_Protection:USBLC6-2SC6
- J3: value I2C TSL2591 -> I2C TSL2591 #1
Connections:
- net +12V: now also R19.1
- net +3V3: now also J10.2 (Pin_2), J13.2 (Pin_2), R20.1, R21.1, U7.5 (VBUS)
- net AUX1: now also J10.3 (Pin_3)
- net AUX2: now also J10.4 (Pin_4)
- net GND: now also J10.1 (Pin_1), J13.1 (Pin_1), U7.2 (GND)
- net Q1_G: now also R19.2
- net AUX3 renamed SDA2
- net SDA2: now also J13.3 (Pin_3), R20.2, U7.1 (I/O1), U7.6 (I/O1)
- net AUX4 renamed SCL2
- net SCL2: now also J13.4 (Pin_4), R21.2, U7.3 (I/O2), U7.4 (I/O2)
