File: hardware/kicad/SQMeter-Hardware-Travel.kicad_pcb (KiCad board)
At the start: 2 copper layers, 85 x 66 mm, 42 parts, among them J10 AUX, J11 Zero left, J12 Zero right, J13 I2C-2 TSL2591 #2, J2 USB-C 5V, J21 BATTERY, J3 I2C TSL2591 #1, J4 I2C MLX90614, J5 I2C BME280, J6 I2C OLED, J7 GPS, SW3 POWER, U4 USBLC6-2SC6, U7 USBLC6-2SC6, U8 MCP73871-2CA

Commit message: feat(travel): 1S2P 18650 support, fuel gauge and cell protection
- MCP73871 in adapter mode, 833 mA charge, safety timer off (7 Ah pack)
- MAX17048 fuel gauge on I2C (0x36): SoC %, voltage, charge/discharge rate;
  ALRT on GPIO1 (replaces the ADC divider)
- DW01A + 2x AO3400A low-side protection for bare cells
- thermal-via QFN for the charger; project symbol library for the MAX17048
Parts:
- removed C18: 100n, Capacitor_SMD:C_0603_1608Metric
- removed R31, R32: 100k, Resistor_SMD:R_0603_1608Metric
- added C21: 100n, Capacitor_SMD:C_0603_1608Metric, F.Cu at (167.0, 119.5)
- added C22: 100n, Capacitor_SMD:C_0603_1608Metric, F.Cu at (167.0, 112.0)
- added Q2: AO3400A, Package_TO_SOT_SMD:SOT-23, F.Cu at (166.5, 124.5)
- added Q3: AO3400A, Package_TO_SOT_SMD:SOT-23, F.Cu at (171.0, 124.5)
- added R33: 100, Resistor_SMD:R_0603_1608Metric, F.Cu at (163.5, 119.5)
- added R34: 1k, Resistor_SMD:R_0603_1608Metric, F.Cu at (175.0, 120.0)
- added R35: 10k, Resistor_SMD:R_0603_1608Metric, F.Cu at (160.0, 112.0)
- added R36: 0, Resistor_SMD:R_0603_1608Metric, F.Cu at (163.5, 115.5)
- added U10: DW01A, Package_TO_SOT_SMD:SOT-23-6, F.Cu at (170.5, 119.5)
- added U11: MAX17048, Package_DFN_QFN:TDFN-8-1EP_2x2mm_P0.5mm_EP0.8x1.2mm, F.Cu at (163.5, 112.0)
- R26: value 2k -> 1.2k
- R27: value 20k -> 10k
- U8: footprint Package_DFN_QFN:QFN-20-1EP_4x4mm_P0.5mm_EP2.5x2.5mm -> Package_DFN_QFN:QFN-20-1EP_4x4mm_P0.5mm_EP2.5x2.5mm_ThermalVias
- moved J21 8.00 mm to (176.0, 132.0)
- moved TH1 2.55 mm to (164.5, 128.5)
Connections:
- J11 pad 4: /VBAT_ADC -> /BAT_ALRT
- J21 pad 2: GND -> /BAT_N
- U8 pad 3: GND -> VBUS
- U8 pad 9: GND -> VBUS
Routing:
- net /BAT_ALRT: track 0.00 -> 55.6 mm, vias 0 -> 2
- net /BAT_N: track 0.00 -> 35.7 mm
- net /VBAT: track 74.1 -> 48.5 mm
- net /VBAT_ADC: track 23.5 -> 0.00 mm
- net VBUS: track 33.3 -> 51.6 mm, vias 0 -> 2
- net /DW_VCC: track 0.00 -> 17.9 mm, vias 0 -> 2
- net /SCL2: track 78.9 -> 63.1 mm
- net /SCL: track 143.1 -> 158.6 mm
- net /SDA: track 142.6 -> 156.3 mm, vias 1 -> 0
- net /DW_CS: track 0.00 -> 12.8 mm, vias 0 -> 2
- net +3V3: track 218.6 -> 229.8 mm, vias 1 -> 4
- net /GAUGE_V: track 0.00 -> 9.20 mm
- net /DW_OD: track 0.00 -> 6.83 mm
- net /GPS_TXO: track 21.0 -> 27.5 mm
- net /BAT_FD: track 0.00 -> 4.50 mm
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Other:
- board text added: "1S BATTERY"
- board text added: "BAT-"
- board text removed: "BATTERY"
