File: hardware/kicad/SQMeter-Hardware-Travel.kicad_sch (KiCad schematic)
At the start: 42 parts, among them J10 AUX, J11 Zero left, J12 Zero right, J13 I2C-2 TSL2591 #2, J2 USB-C 5V, J21 BATTERY, J3 I2C TSL2591 #1, J4 I2C MLX90614, J5 I2C BME280, J6 I2C OLED, J7 GPS, SW3 POWER, U4 USBLC6-2SC6, U7 USBLC6-2SC6, U8 MCP73871-2CA

Commit message: feat(travel): 1S2P 18650 support, fuel gauge and cell protection
- MCP73871 in adapter mode, 833 mA charge, safety timer off (7 Ah pack)
- MAX17048 fuel gauge on I2C (0x36): SoC %, voltage, charge/discharge rate;
  ALRT on GPIO1 (replaces the ADC divider)
- DW01A + 2x AO3400A low-side protection for bare cells
- thermal-via QFN for the charger; project symbol library for the MAX17048
Parts:
- removed C18: 100n, Capacitor_SMD:C_0603_1608Metric, symbol Device:C
- removed D3: SS34, Diode_SMD:D_SMA, symbol Device:D_Schottky
- removed J12: Zero right, Connector_PinSocket_2.54mm:PinSocket_1x09_P2.54mm_Vertical, symbol Connector_Generic:Conn_01x09
- removed R30: 10k, Resistor_SMD:R_0603_1608Metric, symbol Device:R
- removed R32: 100k, Resistor_SMD:R_0603_1608Metric, symbol Device:R
- removed U7: USBLC6-2SC6, Package_TO_SOT_SMD:SOT-23-6, symbol Power_Protection:USBLC6-2SC6
- added C21, C22: 100n, Capacitor_SMD:C_0603_1608Metric, symbol Device:C
- added H2: M3, MountingHole:MountingHole_3.2mm_M3, symbol Mechanical:MountingHole
- added J3: I2C TSL2591 #1, Connector_JST:JST_XH_B4B-XH-A_1x04_P2.50mm_Vertical, symbol Connector_Generic:Conn_01x04
- added J5: I2C BME280, Connector_JST:JST_XH_B4B-XH-A_1x04_P2.50mm_Vertical, symbol Connector_Generic:Conn_01x04
- added Q3: AO3400A, Package_TO_SOT_SMD:SOT-23, symbol Transistor_FET:AO3400A
- added R21: 4.7k, Resistor_SMD:R_0603_1608Metric, symbol Device:R
- added R33: 100, Resistor_SMD:R_0603_1608Metric, symbol Device:R
- added R34: 1k, Resistor_SMD:R_0603_1608Metric, symbol Device:R
- added R35: 10k, Resistor_SMD:R_0603_1608Metric, symbol Device:R
- added R36: 0, Resistor_SMD:R_0603_1608Metric, symbol Device:R
- added U10: DW01A, Package_TO_SOT_SMD:SOT-23-6, symbol Battery_Management:DW01A
- added U11: MAX17048, Package_DFN_QFN:TDFN-8-1EP_2x2mm_P0.5mm_EP0.8x1.2mm, symbol SQMeter:MAX17048
- D3: renamed from J3; value I2C TSL2591 #1 -> SS34; footprint Connector_JST:JST_XH_B4B-XH-A_1x04_P2.50mm_Vertical -> Diode_SMD:D_SMA; symbol Connector_Generic:Conn_01x04 -> Device:D_Schottky; LCSC C144395 -> C8678
- J12: renamed from R21; value 4.7k -> Zero right; footprint Resistor_SMD:R_0603_1608Metric -> Connector_PinSocket_2.54mm:PinSocket_1x09_P2.54mm_Vertical; symbol Device:R -> Connector_Generic:Conn_01x09; LCSC C23162 -> C22438159
- Q2: renamed from R31; value 100k -> AO3400A; footprint Resistor_SMD:R_0603_1608Metric -> Package_TO_SOT_SMD:SOT-23; symbol Device:R -> Transistor_FET:AO3400A; LCSC C25803 -> C20917
- R26: value 2k -> 1.2k; LCSC C22975 -> C22765
- R27: value 20k -> 10k; LCSC C4184 -> C25804
- R30: renamed from J5; value I2C BME280 -> 10k; footprint Connector_JST:JST_XH_B4B-XH-A_1x04_P2.50mm_Vertical -> Resistor_SMD:R_0603_1608Metric; symbol Connector_Generic:Conn_01x04 -> Device:R; LCSC C144395 -> C25804
- U7: renamed from H2; value M3 -> USBLC6-2SC6; footprint MountingHole:MountingHole_3.2mm_M3 -> Package_TO_SOT_SMD:SOT-23-6; symbol Mechanical:MountingHole -> Power_Protection:USBLC6-2SC6; LCSC (none) -> C7519
- U8: footprint Package_DFN_QFN:QFN-20-1EP_4x4mm_P0.5mm_EP2.5x2.5mm -> Package_DFN_QFN:QFN-20-1EP_4x4mm_P0.5mm_EP2.5x2.5mm_ThermalVias
Connections:
- net +3V3: now also R30.1, U7.5 (VBUS), J3.2 (Pin_2), J5.2 (Pin_2), R21.1, R35.1; no longer D3.2 (Pin_2), J12.1, R30.2 (Pin_2)
- net AUX2: now also J12.9 (Pin_9)
- net CHG_PG: now also R30.2
- net DK_5V: now also D3.1 (K)
- net GND: now also U7.2 (GND), C22.2, J3.1 (Pin_1), J5.1 (Pin_1), Q3.2 (S), R34.2, U11.1 (CTG), U11.4 (GND), U11.6 (QSTRT), U11.9 (EP); no longer D3.1 (Pin_1), J21.2 (Pin_2), R30.1 (Pin_1), U8.3 (SEL), U8.9 (~{TE})
- net GPS_RX: now also J12.3 (Pin_3)
- net GPS_TX: now also J12.4 (Pin_4)
- net SCL: now also J12.7 (Pin_7), J3.4 (Pin_4), J5.4 (Pin_4), U11.7 (SCL); no longer D3.4 (Pin_4), R30.4 (Pin_4)
- net SCL2: now also J12.5 (Pin_5), U7.3 (I/O2), U7.4 (I/O2), R21.2; no longer J12.2
- net SDA: now also J12.8 (Pin_8), J3.3 (Pin_3), J5.3 (Pin_3), U11.8 (SDA); no longer D3.3 (Pin_3), R30.3 (Pin_3)
- net SDA2: now also J12.6 (Pin_6), U7.1 (I/O1), U7.6 (I/O1)
- net SYS_SW: now also D3.2 (A)
- net VBAT: now also R33.1, R36.1; no longer Q2.1
- net VBUS: now also U8.3 (SEL), U8.9 (~{TE})
- net VBAT_ADC renamed BAT_ALRT
- net BAT_ALRT: now also R35.2, U11.5 (~{ALRT}); no longer Q2.2
- new net BAT_FD: Q2.3 (D), Q3.3 (D)
- new net BAT_N: C21.2, J21.2 (Pin_2), Q2.2 (S), U10.6 (GND)
- new net DW_CS: R34.1, U10.2 (CS)
- new net DW_OC: Q3.1 (G), U10.3 (OC)
- new net DW_OD: Q2.1 (G), U10.1 (OD)
- new net DW_VCC: C21.1, R33.2, U10.5 (VCC)
- new net GAUGE_V: C22.1, R36.2, U11.2 (CELL), U11.3 (VDD)
- no-connect marks 10 -> 11
